File: hardware/Palm.sch (KiCad schematic (older format))
At the start: 3 parts, among them U1 Adafruit_nRF52_Feather, U2 VEML6075_breakout

Commit message: [design] Add resistors to RGB LED
Parts:
- added R1, R2, R3: 1k, symbol Device:R_Small
- gave numbers to parts that had none: 1
Connections:
- wire segments 19 -> 22
Changed lines of the file:
@@
 EESchema Schematic File Version 4
-LIBS:Palm-cache
 EELAYER 29 0
 EELAYER END
@@
 NoConn ~ 5250 1900
 $Comp
-L Device:LED_BARG D?
+L Device:LED_BARG D1
 U 1 1 5CED4526
 P 7950 2700
-F 0 "D?" H 7950 3197 50  0000 C CNN
-F 1 "LED_BARG" H 7950 3106 50  0000 C CNN
+F 0 "D1" H 7950 3100 50  0000 C CNN
+F 1 "LED_BARG" H 7950 2350 50  0000 C CNN
 F 2 "" H 7950 2650 50  0001 C CNN
 F 3 "~" H 7950 2650 50  0001 C CNN
@@
 Wire Wire Line
 	5050 2300 5250 2300
-Text Label 7600 2500 2    50   ~ 0
+Text Label 7250 2500 2    50   ~ 0
 RED
-Text Label 7600 2700 2    50   ~ 0
+Text Label 7250 2700 2    50   ~ 0
 GREEN
-Text Label 7600 2900 2    50   ~ 0
+Text Label 7250 2900 2    50   ~ 0
 BLUE
 Text Label 8300 2700 0    50   ~ 0
@@
 Wire Wire Line
 	8150 2700 8300 2700
+$Comp
+L Device:R_Small R1
+U 1 1 5CED0CF7
+P 7500 2500
+F 0 "R1" V 7400 2400 50  0000 C CNN
+F 1 "1k" V 7400 2600 50  0000 C CNN
+F 2 "" H 7500 2500 50  0001 C CNN
+F 3 "~" H 7500 2500 50  0001 C CNN
+	1    7500 2500
+	0    1    1    0
+$EndComp
+$Comp
+L Device:R_Small R2
+U 1 1 5CED2FDB
+P 7500 2700
+F 0 "R2" V 7400 2600 50  0000 C CNN
+F 1 "1k" V 7400 2800 50  0000 C CNN
+F 2 "" H 7500 2700 50  0001 C CNN
+F 3 "~" H 7500 2700 50  0001 C CNN
+	1    7500 2700
+	0    1    1    0
+$EndComp
+$Comp
+L Device:R_Small R3
+U 1 1 5CED3479
+P 7500 2900
+F 0 "R3" V 7400 2800 50  0000 C CNN
+F 1 "1k" V 7400 3000 50  0000 C CNN
+F 2 "" H 7500 2900 50  0001 C CNN
+F 3 "~" H 7500 2900 50  0001 C CNN
+	1    7500 2900
+	0    1    1    0
+$EndComp
+Wire Wire Line
+	7250 2500 7400 2500
+Wire Wire Line
+	7250 2700 7400 2700
+Wire Wire Line
+	7250 2900 7400 2900
 $EndSCHEMATC

Commit message: [design] Add 2 switches to on/off power and airplane mode
Parts:
- added J1: Conn_01x02_Female, symbol Connector:Conn_01x02_Female
- added R4: 0R, symbol Device:R_Small
- added R5: 1k, symbol Device:R_Small
- added SW1, SW2: SW_SPST, symbol Switch:SW_SPST
Connections:
- net labels added: EN_SENSOR
- wire segments 22 -> 33
- no-connect marks 21 -> 18
Other:
- note added: "Color display for RGB LED:\nNo color: UV Index 0 - 2\nYellow: UV Index 3 - 5\nOrange: UV Index 6 - 7\nRed: UV Index 8 - 10\nPurple: UV Index 11+\n"
- note added: "JST-PH2 connector \nfor LiPo"
- moved on the sheet: U1, U2

Commit message: [design] Add P-channel MOSFET switch and RGB LED
Co-authored-by: Chinmay Pendharkar <notthetup@gmail.com>
Parts:
- removed R4: 0R, symbol Device:R_Small
- added Q1: IRLML6402, Package_TO_SOT_SMD:SOT-23, symbol Transistor_FET:IRLML6402
- D1: symbol Device:LED_BARG -> Device:LED_RGB
Connections:
- net labels added: +3V3
- net labels removed: 3V
- wire segments 33 -> 38
Other:
- moved on the sheet: U2
Changed lines of the file:
@@
 F 1 "Adafruit_nRF52_Feather" H 3000 1450 50  0000 C CNN
 F 2 "" H 2400 2250 50  0001 C CNN
-F 3 "" H 2400 2250 50  0001 C CNN
+F 3 "https://cdn-learn.adafruit.com/assets/assets/000/052/793/original/microcontrollers_revgsch.png?1523067417" H 2400 2250 50  0001 C CNN
 	1    2550 2400
 	-1   0    0    -1
@@
 	2700 3350 2700 3500
 $Bitmap
-Pos 6350 2150
+Pos 6300 2200
 Scale 0.500000
 Data
@@
 L Sensor_UV:VEML6075_breakout U2
 U 1 1 5CAF1352
-P 9600 1400
-F 0 "U2" H 9900 1650 50  0000 R CNN
-F 1 "VEML6075_breakout" H 9950 950 50  0000 R CNN
-F 2 "" H 9600 1400 50  0001 C CNN
-F 3 "" H 9600 1400 50  0001 C CNN
-	1    9600 1400
+P 9200 1850
+F 0 "U2" H 9500 2100 50  0000 R CNN
+F 1 "VEML6075_breakout" H 8900 1850 50  0000 R CNN
+F 2 "" H 9200 1850 50  0001 C CNN
+F 3 "https://learn.adafruit.com/assets/62587" H 9200 1850 50  0001 C CNN
+	1    9200 1850
 	-1   0    0    -1
 $EndComp
@@
 NoConn ~ 3100 2650
 NoConn ~ 3100 2750
-NoConn ~ 9500 1100
+NoConn ~ 9100 1550
 Wire Wire Line
-	9700 1700 9700 1750
-Wire Wire Line
-	9700 1750 9900 1750
-Text Label 9900 1750 0    50   ~ 0
-GND
+	9300 2150 9300 2200
 Text Label 3300 1950 0    50   ~ 0
 SDA
 Text Label 3300 2050 0    50   ~ 0
 SCL
-Text Label 9100 1450 2    50   ~ 0
+Text Label 8700 1900 2    50   ~ 0
 SCL
-Text Label 9100 1550 2    50   ~ 0
+Text Label 8700 2000 2    50   ~ 0
 SDA
 Wire Wire Line
@@
 	3100 2050 3300 2050
 Wire Wire Line
-	9100 1450 9250 1450
+	8700 1900 8850 1900
 Wire Wire Line
-	9100 1550 9250 1550
+	8700 2000 8850 2000
 Wire Wire Line
 	2600 1050 2600 1300
@@
 NoConn ~ 2000 2100
 $Comp
-L Device:LED_BARG D1
+L Device:LED_RGB D1
 U 1 1 5CED4526
-P 9750 2550
-F 0 "D1" H 9750 2950 50  0000 C CNN
-F 1 "LED_BARG" H 9750 2200 50  0000 C CNN
-F 2 "" H 9750 2500 50  0001 C CNN
-F 3 "~" H 9750 2500 50  0001 C CNN
-	1    9750 2550
+P 9200 3100
+F 0 "D1" H 9200 3500 50  0000 C CNN
+F 1 "LED_BARG" H 9200 2750 50  0000 C CNN
+F 2 "" H 9200 3050 50  0001 C CNN
+F 3 "https://docs-apac.rs-online.com/webdocs/1524/0900766b815247fa.pdf" H 9200 3050 50  0001 C CNN
+	1    9200 3100
 	1    0    0    -1
 $EndComp
@@
 Wire Wire Line
 	1800 2500 2000 2500
-Text Label 9050 2350 2    50   ~ 0
+Text Label 9550 2900 0    50   ~ 0
 RED
-Text Label 9050 2550 2    50   ~ 0
+Text Label 9550 3100 0    50   ~ 0
 GREEN
-Text Label 9050 2750 2    50   ~ 0
+Text Label 9550 3300 0    50   ~ 0
 BLUE
-Text Label 10100 2550 0    50   ~ 0
-GND
 Wire Wire Line
-	9400 2350 9550 2350
+	8850 2900 9000 2900
 Wire Wire Line
-	9400 2550 9550 2550
+	8850 3100 9000 3100
 Wire Wire Line
-	9400 2750 9550 2750
+	8850 3300 9000 3300
 Wire Wire Line
-	9950 2550 10100 2550
+	9400 3100 9550 3100
 $Comp
 L Device:R_Small R1
 U 1 1 5CED0CF7
-P 9300 2350
-F 0 "R1" V 9200 2250 50  0000 C CNN
-F 1 "1k" V 9200 2450 50  0000 C CNN
-F 2 "" H 9300 2350 50  0001 C CNN
-F 3 "~" H 9300 2350 50  0001 C CNN
-	1    9300 2350
+P 8750 2900
+F 0 "R1" V 8650 2800 50  0000 C CNN
+F 1 "1k" V 8650 3000 50  0000 C CNN
+F 2 "" H 8750 2900 50  0001 C CNN
+F 3 "~" H 8750 2900 50  0001 C CNN
+	1    8750 2900
 	0    1    1    0
 $EndComp
@@
 L Device:R_Small R2
 U 1 1 5CED2FDB
-P 9300 2550
-F 0 "R2" V 9200 2450 50  0000 C CNN
-F 1 "1k" V 9200 2650 50  0000 C CNN
-F 2 "" H 9300 2550 50  0001 C CNN
-F 3 "~" H 9300 2550 50  0001 C CNN
-	1    9300 2550
+P 8750 3100
+F 0 "R2" V 8650 3000 50  0000 C CNN
+F 1 "1k" V 8650 3200 50  0000 C CNN
+F 2 "" H 8750 3100 50  0001 C CNN
+F 3 "~" H 8750 3100 50  0001 C CNN
+	1    8750 3100
 	0    1    1    0
 $EndComp
@@
 L Device:R_Small R3
 U 1 1 5CED3479
-P 9300 2750
-F 0 "R3" V 9200 2650 50  0000 C CNN
-F 1 "1k" V 9200 2850 50  0000 C CNN
-F 2 "" H 9300 2750 50  0001 C CNN
-F 3 "~" H 9300 2750 50  0001 C CNN
-	1    9300 2750
+P 8750 3300
+F 0 "R3" V 8650 3200 50  0000 C CNN
+F 1 "1k" V 8650 3400 50  0000 C CNN
+F 2 "" H 8750 3300 50  0001 C CNN
+F 3 "~" H 8750 3300 50  0001 C CNN
+	1    8750 3300
 	0    1    1    0
 $EndComp
 Wire Wire Line
-	9050 2350 9200 2350
+	8500 2900 8650 2900
 Wire Wire Line
-	9050 2550 9200 2550
+	8500 3100 8650 3100
 Wire Wire Line
-	9050 2750 9200 2750
-Text Notes 9150 3550 0    50   ~ 0
+	8500 3300 8650 3300
+Text Notes 9900 3300 0    50   ~ 0
 Color display for RGB LED:\nNo color: UV Index 0 - 2\nYellow: UV Index 3 - 5\nOrange: UV Index 6 - 7\nRed: UV Index 8 - 10\nPurple: UV Index 11+\n
 $Comp
@@
 	1800 1300 1800 1450
 Wire Wire Line
-	9700 1000 9700 1100
-Connection ~ 9700 1000
-$Comp
-L Device:R_Small R4
-U 1 1 5CF42FD9
-P 9800 1000
-F 0 "R4" V 9700 1000 50  0000 C CNN
-F 1 "0R" V 9900 1000 50  0000 C CNN
-F 2 "" H 9800 1000 50  0001 C CNN
-F 3 "~" H 9800 1000 50  0001 C CNN
-	1    9800 1000
-	0    1    1    0
-$EndComp
+	9300 1450 9300 1500
 Text Label 3250 2850 0    50   ~ 0
 EN_SENSOR
 Wire Wire Line
 	3100 2850 3250 2850
-Text Label 10100 1000 0    50   ~ 0
+Text Label 8850 1250 2    50   ~ 0
 EN_SENSOR
-Wire Wire Line
-	9900 1000 10100 1000
 $Comp
 L Switch:SW_SPST SW2
@@
 	1    0    0    -1
 $EndComp
-Text Label 2350 3050 2    50   ~ 0
-3V
-Text Label 4200 2950 0    50   ~ 0
-3V
 Wire Wire Line
 	1850 3050 2000 3050
@@
 	4050 2950 4200 2950
 $Comp
+L Transistor_FET:IRLML6402 Q1
+U 1 1 5CF39500
+P 9200 1250
+F 0 "Q1" H 9406 1204 50  0000 L CNN
+F 1 "IRLML6402" H 9406 1295 50  0000 L CNN
+F 2 "Package_TO_SOT_SMD:SOT-23" H 9400 1175 50  0001 L CIN
+F 3 "https://docs-apac.rs-online.com/webdocs/10c7/0900766b810c708d.pdf" H 9200 1250 50  0001 L CNN
+	1    9200 1250
+	1    0    0    1
+$EndComp
+Wire Wire Line
+	8850 1250 9000 1250
+$Comp
+L power:+3V3 #PWR03
+U 1 1 5CF46C12
+P 1850 3050
+F 0 "#PWR03" H 1850 2900 50  0001 C CNN
+F 1 "+3V3" H 1865 3223 50  0000 C CNN
+F 2 "" H 1850 3050 50  0001 C CNN
+F 3 "" H 1850 3050 50  0001 C CNN
+	1    1850 3050
+	1    0    0    -1
+$EndComp
+$Comp
+L power:+3V3 #PWR04
+U 1 1 5CF47131
+P 9300 1050
+F 0 "#PWR04" H 9300 900 50  0001 C CNN
+F 1 "+3V3" H 9315 1223 50  0000 C CNN
+F 2 "" H 9300 1050 50  0001 C CNN
+F 3 "" H 9300 1050 50  0001 C CNN
+	1    9300 1050
+	1    0    0    -1
+$EndComp
+$Comp
 L power:PWR_FLAG #FLG0103
-U 1 1 5CF44D78
-P 9700 1000
-F 0 "#FLG0103" H 9700 1075 50  0001 C CNN
-F 1 "PWR_FLAG" V 9700 1300 50  0000 C CNN
-F 2 "" H 9700 1000 50  0001 C CNN
-F 3 "~" H 9700 1000 50  0001 C CNN
-	1    9700 1000
-	0    -1   -1   0
+U 1 1 5CF47E2F
+P 9300 1500
+F 0 "#FLG0103" H 9300 1575 50  0001 C CNN
+F 1 "PWR_FLAG" V 9300 1800 50  0000 C CNN
+F 2 "" H 9300 1500 50  0001 C CNN
+F 3 "~" H 9300 1500 50  0001 C CNN
+	1    9300 1500
+	0    1    1    0
+$EndComp
+Connection ~ 9300 1500
+Wire Wire Line
+	9300 1500 9300 1550
+$Comp
+L power:+3V3 #PWR0103
+U 1 1 5CF48BA3
+P 4200 2950
+F 0 "#PWR0103" H 4200 2800 50  0001 C CNN
+F 1 "+3V3" H 4215 3123 50  0000 C CNN
+F 2 "" H 4200 2950 50  0001 C CNN
+F 3 "" H 4200 2950 50  0001 C CNN
+	1    4200 2950
+	1    0    0    -1
+$EndComp
+Wire Wire Line
+	9400 2900 9550 2900
+Wire Wire Line
+	9400 3300 9550 3300
+$Comp
+L power:GND #PWR0104
+U 1 1 5CF56626
+P 9300 2200
+F 0 "#PWR0104" H 9300 1950 50  0001 C CNN
+F 1 "GND" H 9305 2027 50  0000 C CNN
+F 2 "" H 9300 2200 50  0001 C CNN
+F 3 "" H 9300 2200 50  0001 C CNN
+	1    9300 2200
+	1    0    0    -1
+$EndComp
+$Comp
+L power:GND #PWR0105
+U 1 1 5CF5940C
+P 8500 3450
+F 0 "#PWR0105" H 8500 3200 50  0001 C CNN
+F 1 "GND" H 8505 3277 50  0000 C CNN
+F 2 "" H 8500 3450 50  0001 C CNN
+F 3 "" H 8500 3450 50  0001 C CNN
+	1    8500 3450
+	1    0    0    -1
 $EndComp
-Text Label 1850 3050 2    50   ~ 0
-3V
+Wire Wire Line
+	8500 2900 8500 3100
+Connection ~ 8500 3100
+Wire Wire Line
+	8500 3100 8500 3300
+Connection ~ 8500 3300
+Wire Wire Line
+	8500 3300 8500 3450
 $EndSCHEMATC
