File: hardware/Palm.sch (KiCad schematic (older format))
At the start: 11 parts, among them J1 Conn_01x02_Female, Q1 IRLML6402, SW1 SW_SPST, SW2 SW_SPST, U1 Adafruit_nRF52_Feather, U2 VEML6075_breakout

Commit message: [design] Add information on vendor, manufacturer, part no, package
Parts:
- D1: Manufacturer (none) -> Cree; Package (none) -> SMD; Part No. (none) -> SLV6A-FKB-CK1P1G1BB7R3R3; Vendor (none) -> RS Components
- J1, SW1, SW2: Package (none) -> SMD; Vendor (none) -> AliExpress
- Q1: Manufacturer (none) -> Infineon; Package (none) -> SOT-23; Part No. (none) -> IRLML2246TRPBF; Vendor (none) -> RS Components
- R1, R2, R3, R5: Package (none) -> 0805; Stock (none) -> 18-res-0805-1k
- U1: Manufacturer (none) -> Adafruit; Package (none) -> TH; Part No. (none) -> 3406; Vendor (none) -> Adafruit
- U2: Manufacturer (none) -> Adafruit; Package (none) -> TH; Part No. (none) -> 3964; Vendor (none) -> Adafruit
Changed lines of the file:
@@
 F 2 "" H 2400 2250 50  0001 C CNN
 F 3 "https://cdn-learn.adafruit.com/assets/assets/000/052/793/original/microcontrollers_revgsch.png?1523067417" H 2400 2250 50  0001 C CNN
+F 4 "Adafruit" H 0   0   50  0001 C CNN "Manufacturer"
+F 5 "TH" H 0   0   50  0001 C CNN "Package"
+F 6 "3406" H 0   0   50  0001 C CNN "Part No."
+F 7 "Adafruit" H 0   0   50  0001 C CNN "Vendor"
 	1    2550 2400
 	-1   0    0    -1
@@
 F 2 "" H 9200 1850 50  0001 C CNN
 F 3 "https://learn.adafruit.com/assets/62587" H 9200 1850 50  0001 C CNN
+F 4 "Adafruit" H 0   0   50  0001 C CNN "Manufacturer"
+F 5 "TH" H 0   0   50  0001 C CNN "Package"
+F 6 "3964" H 0   0   50  0001 C CNN "Part No."
+F 7 "Adafruit" H 0   0   50  0001 C CNN "Vendor"
 	1    9200 1850
 	-1   0    0    -1
@@
 F 2 "" H 9200 3050 50  0001 C CNN
 F 3 "https://docs-apac.rs-online.com/webdocs/1524/0900766b815247fa.pdf" H 9200 3050 50  0001 C CNN
+F 4 "Cree" H 0   0   50  0001 C CNN "Manufacturer"
+F 5 "SMD" H 0   0   50  0001 C CNN "Package"
+F 6 "SLV6A-FKB-CK1P1G1BB7R3R3 " H 0   0   50  0001 C CNN "Part No."
+F 7 "RS Components" H 0   0   50  0001 C CNN "Vendor"
 	1    9200 3100
 	1    0    0    -1
@@
 F 2 "" H 8750 2900 50  0001 C CNN
 F 3 "~" H 8750 2900 50  0001 C CNN
+F 4 "0805" H 0   0   50  0001 C CNN "Package"
+F 5 "18-res-0805-1k" H 0   0   50  0001 C CNN "Stock"
 	1    8750 2900
 	0    1    1    0
@@
 F 2 "" H 8750 3100 50  0001 C CNN
 F 3 "~" H 8750 3100 50  0001 C CNN
+F 4 "0805" H 0   0   50  0001 C CNN "Package"
+F 5 "18-res-0805-1k" H 0   0   50  0001 C CNN "Stock"
 	1    8750 3100
 	0    1    1    0
@@
 F 2 "" H 8750 3300 50  0001 C CNN
 F 3 "~" H 8750 3300 50  0001 C CNN
+F 4 "0805" H 0   0   50  0001 C CNN "Package"
+F 5 "18-res-0805-1k" H 0   0   50  0001 C CNN "Stock"
 	1    8750 3300
 	0    1    1    0
@@
 F 1 "SW_SPST" H 2050 1344 50  0000 C CNN
 F 2 "" H 2050 1200 50  0001 C CNN
-F 3 "~" H 2050 1200 50  0001 C CNN
+F 3 "https://www.aliexpress.com/item/50Pcs-Mini-7-Pin-On-Off-1P2T-SPDT-MSK-12C02-SMD-Toggle-Slide-Switch-For-MP3/32856542440.html" H 2050 1200 50  0001 C CNN
+F 4 "SMD" H 0   0   50  0001 C CNN "Package"
+F 5 "AliExpress" H 0   0   50  0001 C CNN "Vendor"
 	1    2050 1200
 	-1   0    0    -1
@@
 F 2 "" H 1500 1200 50  0001 C CNN
 F 3 "~" H 1500 1200 50  0001 C CNN
+F 4 "SMD" H 0   0   50  0001 C CNN "Package"
+F 5 "AliExpress" H 0   0   50  0001 C CNN "Vendor"
 	1    1500 1200
 	-1   0    0    -1
@@
 F 1 "SW_SPST" H 3850 2850 50  0000 C CNN
 F 2 "" H 3850 2950 50  0001 C CNN
-F 3 "~" H 3850 2950 50  0001 C CNN
+F 3 "https://www.aliexpress.com/item/50Pcs-Mini-7-Pin-On-Off-1P2T-SPDT-MSK-12C02-SMD-Toggle-Slide-Switch-For-MP3/32856542440.html" H 3850 2950 50  0001 C CNN
+F 4 "SMD" H 0   0   50  0001 C CNN "Package"
+F 5 "AliExpress" H 0   0   50  0001 C CNN "Vendor"
 	1    3850 2950
 	1    0    0    -1
@@
 F 2 "" H 3450 3150 50  0001 C CNN
 F 3 "~" H 3450 3150 50  0001 C CNN
+F 4 "0805" H 0   0   50  0001 C CNN "Package"
+F 5 "18-res-0805-1k" H 0   0   50  0001 C CNN "Stock"
 	1    3450 3150
 	1    0    0    -1
@@
 F 2 "Package_TO_SOT_SMD:SOT-23" H 9400 1175 50  0001 L CIN
 F 3 "https://docs-apac.rs-online.com/webdocs/10c7/0900766b810c708d.pdf" H 9200 1250 50  0001 L CNN
+F 4 "Infineon" H 0   0   50  0001 C CNN "Manufacturer"
+F 5 "SOT-23" H 0   0   50  0001 C CNN "Package"
+F 6 "IRLML2246TRPBF" H 0   0   50  0001 C CNN "Part No."
+F 7 "RS Components" H 0   0   50  0001 C CNN "Vendor"
 	1    9200 1250
 	1    0    0    1

Commit message: [bom] Generate bill of materials
Parts:
- removed R5: 1k, symbol Device:R_Small
- D1: Minimum Order (none) -> 10; Unit cost (none) -> 0.632; Vendor link (none) -> https://sg.rs-online.com/web/p/products/1238680/
- J1: Manufacturer (none) -> JST; Minimum Order (none) -> 5; Part No. (none) -> B2B-PH-SM4-TB(LF)(SN); Unit cost (none) -> 0.486; Vendor AliExpress -> RS Components; Vendor link (none) -> https://sg.rs-online.com/web/p/pcb-headers/6881325/
- Q1: Minimum Order (none) -> 5; Unit cost (none) -> 0.224; Vendor link (none) -> https://sg.rs-online.com/web/p/products/7604432/
- R1, R2, R3: footprint (none) -> Resistor_SMD:R_0805_2012Metric_Pad1.15x1.40mm_HandSolder; Minimum Order (none) -> 1
- SW1, SW2: value SW_SPST -> SW_SPDT; symbol Switch:SW_SPST -> Switch:SW_SPDT; Minimum Order (none) -> 1; Unit cost (none) -> 1.90; Vendor link (none) -> https://www.aliexpress.com/item/50Pcs-Mini-7-Pin-On-Off-1P2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
- U1: Minimum Order (none) -> 1; Stock (none) -> prototype-4; Unit cost (none) -> 34.0; Vendor link (none) -> https://www.adafruit.com/product/3406
- U2: Minimum Order (none) -> 1; Stock (none) -> prototype-5; Unit cost (none) -> 8.20; Vendor link (none) -> https://www.adafruit.com/product/3964
Connections:
- wire segments 38 -> 37
- no-connect marks 18 -> 19
Changed lines of the file:
@@
 F 6 "3406" H 0   0   50  0001 C CNN "Part No."
 F 7 "Adafruit" H 0   0   50  0001 C CNN "Vendor"
+F 8 "prototype-4" H 0   0   50  0001 C CNN "Stock"
+F 9 "34.0" H 0   0   50  0001 C CNN "Unit cost"
+F 10 "https://www.adafruit.com/product/3406" H 0   0   50  0001 C CNN "Vendor link"
+F 11 "1" H 0   0   50  0001 C CNN "Minimum Order"
 	1    2550 2400
 	-1   0    0    -1
@@
 F 6 "3964" H 0   0   50  0001 C CNN "Part No."
 F 7 "Adafruit" H 0   0   50  0001 C CNN "Vendor"
+F 8 "prototype-5" H 0   0   50  0001 C CNN "Stock"
+F 9 "8.20" H 0   0   50  0001 C CNN "Unit cost"
+F 10 "https://www.adafruit.com/product/3964" H 0   0   50  0001 C CNN "Vendor link"
+F 11 "1" H 0   0   50  0001 C CNN "Minimum Order"
 	1    9200 1850
 	-1   0    0    -1
@@
 F 6 "SLV6A-FKB-CK1P1G1BB7R3R3 " H 0   0   50  0001 C CNN "Part No."
 F 7 "RS Components" H 0   0   50  0001 C CNN "Vendor"
+F 8 "10" H 0   0   50  0001 C CNN "Minimum Order"
+F 9 "0.632" H 0   0   50  0001 C CNN "Unit cost"
+F 10 "https://sg.rs-online.com/web/p/products/1238680/" H 0   0   50  0001 C CNN "Vendor link"
 	1    9200 3100
 	1    0    0    -1
@@
 F 0 "R1" V 8650 2800 50  0000 C CNN
 F 1 "1k" V 8650 3000 50  0000 C CNN
-F 2 "" H 8750 2900 50  0001 C CNN
+F 2 "Resistor_SMD:R_0805_2012Metric_Pad1.15x1.40mm_HandSolder" H 8750 2900 50  0001 C CNN
 F 3 "~" H 8750 2900 50  0001 C CNN
 F 4 "0805" H 0   0   50  0001 C CNN "Package"
 F 5 "18-res-0805-1k" H 0   0   50  0001 C CNN "Stock"
+F 6 "1" H 0   0   50  0001 C CNN "Minimum Order"
 	1    8750 2900
 	0    1    1    0
@@
 F 0 "R2" V 8650 3000 50  0000 C CNN
 F 1 "1k" V 8650 3200 50  0000 C CNN
-F 2 "" H 8750 3100 50  0001 C CNN
+F 2 "Resistor_SMD:R_0805_2012Metric_Pad1.15x1.40mm_HandSolder" H 8750 3100 50  0001 C CNN
 F 3 "~" H 8750 3100 50  0001 C CNN
 F 4 "0805" H 0   0   50  0001 C CNN "Package"
 F 5 "18-res-0805-1k" H 0   0   50  0001 C CNN "Stock"
+F 6 "1" H 0   0   50  0001 C CNN "Minimum Order"
 	1    8750 3100
 	0    1    1    0
@@
 F 0 "R3" V 8650 3200 50  0000 C CNN
 F 1 "1k" V 8650 3400 50  0000 C CNN
-F 2 "" H 8750 3300 50  0001 C CNN
+F 2 "Resistor_SMD:R_0805_2012Metric_Pad1.15x1.40mm_HandSolder" H 8750 3300 50  0001 C CNN
 F 3 "~" H 8750 3300 50  0001 C CNN
 F 4 "0805" H 0   0   50  0001 C CNN "Package"
 F 5 "18-res-0805-1k" H 0   0   50  0001 C CNN "Stock"
+F 6 "1" H 0   0   50  0001 C CNN "Minimum Order"
 	1    8750 3300
 	0    1    1    0
@@
 Color display for RGB LED:\nNo color: UV Index 0 - 2\nYellow: UV Index 3 - 5\nOrange: UV Index 6 - 7\nRed: UV Index 8 - 10\nPurple: UV Index 11+\n
 $Comp
-L Switch:SW_SPST SW1
+L Switch:SW_SPDT SW1
 U 1 1 5CEE5E28
 P 2050 1200
-F 0 "SW1" H 2050 1435 50  0000 C CNN
-F 1 "SW_SPST" H 2050 1344 50  0000 C CNN
+F 0 "SW1" H 2150 1400 50  0000 C CNN
+F 1 "SW_SPDT" H 1900 1300 50  0000 C CNN
 F 2 "" H 2050 1200 50  0001 C CNN
 F 3 "https://www.aliexpress.com/item/50Pcs-Mini-7-Pin-On-Off-1P2T-SPDT-MSK-12C02-SMD-Toggle-Slide-Switch-For-MP3/32856542440.html" H 2050 1200 50  0001 C CNN
 F 4 "SMD" H 0   0   50  0001 C CNN "Package"
 F 5 "AliExpress" H 0   0   50  0001 C CNN "Vendor"
+F 6 "1.90 " H 0   0   50  0001 C CNN "Unit cost"
+F 7 "https://www.aliexpress.com/item/50Pcs-Mini-7-Pin-On-Off-1P2T-SPDT-MSK-12C02-SMD-Toggle-Slide-Switch-For-MP3/32856542440.html" H 0   0   50  0001 C CNN "Vendor link"
+F 8 "1" H 0   0   50  0001 C CNN "Minimum Order"
 	1    2050 1200
 	-1   0    0    -1
@@
 L Connector:Conn_01x02_Female J1
 U 1 1 5CEE767E
-P 1500 1200
-F 0 "J1" H 1528 1176 50  0000 L CNN
-F 1 "Conn_01x02_Female" H 1528 1085 50  0000 L CNN
-F 2 "" H 1500 1200 50  0001 C CNN
-F 3 "~" H 1500 1200 50  0001 C CNN
-F 4 "SMD" H 0   0   50  0001 C CNN "Package"
-F 5 "AliExpress" H 0   0   50  0001 C CNN "Vendor"
-	1    1500 1200
+P 1350 1100
+F 0 "J1" H 1378 1076 50  0000 L CNN
+F 1 "Conn_01x02_Female" H 1378 985 50  0000 L CNN
+F 2 "" H 1350 1100 50  0001 C CNN
+F 3 "https://docs-apac.rs-online.com/webdocs/13ce/0900766b813ce4b4.pdf" H 1350 1100 50  0001 C CNN
+F 4 "SMD" H -150 -100 50  0001 C CNN "Package"
+F 5 "RS Components" H -150 -100 50  0001 C CNN "Vendor"
+F 6 "5" H -150 -100 50  0001 C CNN "Minimum Order"
+F 7 "JST" H 0   0   50  0001 C CNN "Manufacturer"
+F 8 "B2B-PH-SM4-TB(LF)(SN) " H 0   0   50  0001 C CNN "Part No."
+F 9 "0.486" H 0   0   50  0001 C CNN "Unit cost"
+F 10 "https://sg.rs-online.com/web/p/pcb-headers/6881325/" H 0   0   50  0001 C CNN "Vendor link"
+	1    1350 1100
 	-1   0    0    -1
 $EndComp
-Wire Wire Line
-	1850 1200 1700 1200
-Text Notes 1050 1050 0    50   ~ 0
+Text Notes 1050 950  0    50   ~ 0
 JST-PH2 connector \nfor LiPo
 Wire Wire Line
@@
 L power:GND #PWR01
 U 1 1 5CF419F7
-P 1800 1450
-F 0 "#PWR01" H 1800 1200 50  0001 C CNN
-F 1 "GND" H 1805 1277 50  0000 C CNN
-F 2 "" H 1800 1450 50  0001 C CNN
-F 3 "" H 1800 1450 50  0001 C CNN
-	1    1800 1450
+P 1650 1350
+F 0 "#PWR01" H 1650 1100 50  0001 C CNN
+F 1 "GND" H 1655 1177 50  0000 C CNN
+F 2 "" H 1650 1350 50  0001 C CNN
+F 3 "" H 1650 1350 50  0001 C CNN
+	1    1650 1350
 	1    0    0    -1
 $EndComp
 Wire Wire Line
-	1700 1300 1800 1300
+	1550 1200 1650 1200
 Wire Wire Line
-	1800 1300 1800 1450
+	1650 1200 1650 1350
 Wire Wire Line
 	9300 1450 9300 1500
@@
 EN_SENSOR
 $Comp
-L Switch:SW_SPST SW2
+L Switch:SW_SPDT SW2
 U 1 1 5CF4F316
 P 3850 2950
-F 0 "SW2" H 3850 3050 50  0000 C CNN
-F 1 "SW_SPST" H 3850 2850 50  0000 C CNN
+F 0 "SW2" H 3800 2850 50  0000 C CNN
+F 1 "SW_SPDT" H 3750 2750 50  0000 C CNN
 F 2 "" H 3850 2950 50  0001 C CNN
 F 3 "https://www.aliexpress.com/item/50Pcs-Mini-7-Pin-On-Off-1P2T-SPDT-MSK-12C02-SMD-Toggle-Slide-Switch-For-MP3/32856542440.html" H 3850 2950 50  0001 C CNN
 F 4 "SMD" H 0   0   50  0001 C CNN "Package"
 F 5 "AliExpress" H 0   0   50  0001 C CNN "Vendor"
+F 6 "1.90 " H 0   0   50  0001 C CNN "Unit cost"
+F 7 "https://www.aliexpress.com/item/50Pcs-Mini-7-Pin-On-Off-1P2T-SPDT-MSK-12C02-SMD-Toggle-Slide-Switch-For-MP3/32856542440.html" H 0   0   50  0001 C CNN "Vendor link"
+F 8 "1" H 0   0   50  0001 C CNN "Minimum Order"
 	1    3850 2950
 	1    0    0    -1
@@
 	1850 3050 2000 3050
 $Comp
-L Device:R_Small R5
-U 1 1 5CF51E77
-P 3450 3150
-F 0 "R5" H 3300 3150 50  0000 L CNN
-F 1 "1k" H 3500 3150 50  0000 L CNN
-F 2 "" H 3450 3150 50  0001 C CNN
-F 3 "~" H 3450 3150 50  0001 C CNN
-F 4 "0805" H 0   0   50  0001 C CNN "Package"
-F 5 "18-res-0805-1k" H 0   0   50  0001 C CNN "Stock"
-	1    3450 3150
-	1    0    0    -1
-$EndComp
-Wire Wire Line
-	3450 2950 3450 3050
-Wire Wire Line
-	3450 2950 3650 2950
-$Comp
 L power:GND #PWR02
 U 1 1 5CF52DF5
-P 3450 3400
-F 0 "#PWR02" H 3450 3150 50  0001 C CNN
-F 1 "GND" H 3455 3227 50  0000 C CNN
-F 2 "" H 3450 3400 50  0001 C CNN
-F 3 "" H 3450 3400 50  0001 C CNN
-	1    3450 3400
+P 4200 3100
+F 0 "#PWR02" H 4200 2850 50  0001 C CNN
+F 1 "GND" H 4205 2927 50  0000 C CNN
+F 2 "" H 4200 3100 50  0001 C CNN
+F 3 "" H 4200 3100 50  0001 C CNN
+	1    4200 3100
 	1    0    0    -1
 $EndComp
 Wire Wire Line
-	3450 3250 3450 3400
-Wire Wire Line
-	3100 2950 3450 2950
-Connection ~ 3450 2950
-Wire Wire Line
 	2250 1200 2500 1200
 Wire Wire Line
-	4050 2950 4200 2950
+	4050 2850 4200 2850
 $Comp
 L Transistor_FET:IRLML6402 Q1
@@
 F 6 "IRLML2246TRPBF" H 0   0   50  0001 C CNN "Part No."
 F 7 "RS Components" H 0   0   50  0001 C CNN "Vendor"
+F 8 "5" H 0   0   50  0001 C CNN "Minimum Order"
+F 9 "0.224" H 0   0   50  0001 C CNN "Unit cost"
+F 10 "https://sg.rs-online.com/web/p/products/7604432/" H 0   0   50  0001 C CNN "Vendor link"
 	1    9200 1250
 	1    0    0    1
@@
 L power:+3V3 #PWR0103
 U 1 1 5CF48BA3
-P 4200 2950
-F 0 "#PWR0103" H 4200 2800 50  0001 C CNN
-F 1 "+3V3" H 4215 3123 50  0000 C CNN
-F 2 "" H 4200 2950 50  0001 C CNN
-F 3 "" H 4200 2950 50  0001 C CNN
-	1    4200 2950
+P 4200 2850
+F 0 "#PWR0103" H 4200 2700 50  0001 C CNN
+F 1 "+3V3" H 4215 3023 50  0000 C CNN
+F 2 "" H 4200 2850 50  0001 C CNN
+F 3 "" H 4200 2850 50  0001 C CNN
+	1    4200 2850
 	1    0    0    -1
 $EndComp
@@
 Wire Wire Line
 	8500 3300 8500 3450
+Wire Wire Line
+	1550 1100 1850 1100
+NoConn ~ 1850 1300
+Wire Wire Line
+	3100 2950 3650 2950
+Wire Wire Line
+	4200 3050 4200 3100
+Wire Wire Line
+	4050 3050 4200 3050
 $EndSCHEMATC

Commit message: [bom] Add category in BOM generation
Parts:
- D1, Q1, R1, R2, R3, U1, U2: Category (none) -> Electronics
- J1, SW1, SW2: Category (none) -> Connector
Changed lines of the file:
@@
 F 10 "https://www.adafruit.com/product/3406" H 0   0   50  0001 C CNN "Vendor link"
 F 11 "1" H 0   0   50  0001 C CNN "Minimum Order"
+F 12 "Electronics" H 0   0   50  0001 C CNN "Category"
 	1    2550 2400
 	-1   0    0    -1
@@
 F 10 "https://www.adafruit.com/product/3964" H 0   0   50  0001 C CNN "Vendor link"
 F 11 "1" H 0   0   50  0001 C CNN "Minimum Order"
+F 12 "Electronics" H 0   0   50  0001 C CNN "Category"
 	1    9200 1850
 	-1   0    0    -1
@@
 F 9 "0.632" H 0   0   50  0001 C CNN "Unit cost"
 F 10 "https://sg.rs-online.com/web/p/products/1238680/" H 0   0   50  0001 C CNN "Vendor link"
+F 11 "Electronics" H 0   0   50  0001 C CNN "Category"
 	1    9200 3100
 	1    0    0    -1
@@
 F 5 "18-res-0805-1k" H 0   0   50  0001 C CNN "Stock"
 F 6 "1" H 0   0   50  0001 C CNN "Minimum Order"
+F 7 "Electronics" H 0   0   50  0001 C CNN "Category"
 	1    8750 2900
 	0    1    1    0
@@
 F 5 "18-res-0805-1k" H 0   0   50  0001 C CNN "Stock"
 F 6 "1" H 0   0   50  0001 C CNN "Minimum Order"
+F 7 "Electronics" H 0   0   50  0001 C CNN "Category"
 	1    8750 3100
 	0    1    1    0
@@
 F 5 "18-res-0805-1k" H 0   0   50  0001 C CNN "Stock"
 F 6 "1" H 0   0   50  0001 C CNN "Minimum Order"
+F 7 "Electronics" H 0   0   50  0001 C CNN "Category"
 	1    8750 3300
 	0    1    1    0
@@
 F 7 "https://www.aliexpress.com/item/50Pcs-Mini-7-Pin-On-Off-1P2T-SPDT-MSK-12C02-SMD-Toggle-Slide-Switch-For-MP3/32856542440.html" H 0   0   50  0001 C CNN "Vendor link"
 F 8 "1" H 0   0   50  0001 C CNN "Minimum Order"
+F 9 "Connector" H 0   0   50  0001 C CNN "Category"
 	1    2050 1200
 	-1   0    0    -1
@@
 F 9 "0.486" H 0   0   50  0001 C CNN "Unit cost"
 F 10 "https://sg.rs-online.com/web/p/pcb-headers/6881325/" H 0   0   50  0001 C CNN "Vendor link"
+F 11 "Connector" H 0   0   50  0001 C CNN "Category"
 	1    1350 1100
 	-1   0    0    -1
@@
 F 7 "https://www.aliexpress.com/item/50Pcs-Mini-7-Pin-On-Off-1P2T-SPDT-MSK-12C02-SMD-Toggle-Slide-Switch-For-MP3/32856542440.html" H 0   0   50  0001 C CNN "Vendor link"
 F 8 "1" H 0   0   50  0001 C CNN "Minimum Order"
+F 9 "Connector" H 0   0   50  0001 C CNN "Category"
 	1    3850 2950
 	1    0    0    -1
@@
 F 9 "0.224" H 0   0   50  0001 C CNN "Unit cost"
 F 10 "https://sg.rs-online.com/web/p/products/7604432/" H 0   0   50  0001 C CNN "Vendor link"
+F 11 "Electronics" H 0   0   50  0001 C CNN "Category"
 	1    9200 1250
 	1    0    0    1

Commit message: [footprint] Associate nRF52 breakbout board with symbol and footprint
Parts:
- U1: footprint (none) -> nRF52_Bluefruit_Adafruit_breakout:nRF52_Bluefruit_Adafruit_breakout_board
- U2: footprint (none) -> VEML6075_breakout_board:VEML6075_breakout_board
Changed lines of the file:
@@
 F 0 "U1" H 2950 3350 50  0000 C CNN
 F 1 "Adafruit_nRF52_Feather" H 3000 1450 50  0000 C CNN
-F 2 "" H 2400 2250 50  0001 C CNN
+F 2 "nRF52_Bluefruit_Adafruit_breakout:nRF52_Bluefruit_Adafruit_breakout_board" H 2400 2250 50  0001 C CNN
 F 3 "https://cdn-learn.adafruit.com/assets/assets/000/052/793/original/microcontrollers_revgsch.png?1523067417" H 2400 2250 50  0001 C CNN
 F 4 "Adafruit" H 0   0   50  0001 C CNN "Manufacturer"
@@
 F 0 "U2" H 9500 2100 50  0000 R CNN
 F 1 "VEML6075_breakout" H 8900 1850 50  0000 R CNN
-F 2 "" H 9200 1850 50  0001 C CNN
+F 2 "VEML6075_breakout_board:VEML6075_breakout_board" H 9200 1850 50  0001 C CNN
 F 3 "https://learn.adafruit.com/assets/62587" H 9200 1850 50  0001 C CNN
 F 4 "Adafruit" H 0   0   50  0001 C CNN "Manufacturer"
@@
 Wire Wire Line
 	4050 3050 4200 3050
+Entry Wire Line
+	8300 -350 8400 -250
 $EndSCHEMATC

Commit message: [footprint] Associate all symbols with footprint
Parts:
- D1, J1: footprint (none) -> Connector_JST:JST_PH_S2B-PH-K_1x02_P2.00mm_Horizontal
- SW1, SW2: footprint (none) -> Button_Switch_SMD:SW_SPDT_PCM12
Other:
- note added: "RGB LED"
- note added: "UV Sensor"
- note added: "nRF52 breakout board"
- moved on the sheet: U1, U2

Commit message: [footprint] Layout all footprints
Parts:
- D1: footprint Connector_JST:JST_PH_S2B-PH-K_1x02_P2.00mm_Horizontal -> CREE_RGB_LED_-PLCC-6_5.5x5.5mm:LED_RGB_Cree-PLCC-6_5.5x5.5mm_P2.1mm
- J1: footprint Connector_JST:JST_PH_S2B-PH-K_1x02_P2.00mm_Horizontal -> Connector_JST:JST_PH_S2B-PH-SM4-TB_1x02-1MP_P2.00mm_Horizontal
- U2: footprint VEML6075_breakout_board:VEML6075_breakout_board -> veml6075_breakout_board:VEML6075_breakout_board
Changed lines of the file:
@@
 F 0 "U2" H 10100 2150 50  0000 R CNN
 F 1 "VEML6075_breakout" H 9500 1900 50  0000 R CNN
-F 2 "VEML6075_breakout_board:VEML6075_breakout_board" H 9800 1900 50  0001 C CNN
+F 2 "veml6075_breakout_board:VEML6075_breakout_board" H 9800 1900 50  0001 C CNN
 F 3 "https://learn.adafruit.com/assets/62587" H 9800 1900 50  0001 C CNN
 F 4 "Adafruit" H 600 50  50  0001 C CNN "Manufacturer"
@@
 F 0 "D1" H 10300 3500 50  0000 C CNN
 F 1 "LED_BARG" H 10300 2750 50  0000 C CNN
-F 2 "Connector_JST:JST_PH_S2B-PH-K_1x02_P2.00mm_Horizontal" H 10300 3050 50  0001 C CNN
+F 2 "CREE_RGB_LED_-PLCC-6_5.5x5.5mm:LED_RGB_Cree-PLCC-6_5.5x5.5mm_P2.1mm" H 10300 3050 50  0001 C CNN
 F 3 "https://docs-apac.rs-online.com/webdocs/1524/0900766b815247fa.pdf" H 10300 3050 50  0001 C CNN
 F 4 "Cree" H 1100 0   50  0001 C CNN "Manufacturer"
@@
 F 0 "J1" H 1578 1076 50  0000 L CNN
 F 1 "Conn_01x02_Female" H 1578 985 50  0000 L CNN
-F 2 "Connector_JST:JST_PH_S2B-PH-K_1x02_P2.00mm_Horizontal" H 1550 1100 50  0001 C CNN
+F 2 "Connector_JST:JST_PH_S2B-PH-SM4-TB_1x02-1MP_P2.00mm_Horizontal" H 1550 1100 50  0001 C CNN
 F 3 "https://docs-apac.rs-online.com/webdocs/13ce/0900766b813ce4b4.pdf" H 1550 1100 50  0001 C CNN
 F 4 "SMD" H 50  -100 50  0001 C CNN "Package"

Commit message: [footprint] Link SDA/SCL and RGB LED tracks
Changed lines of the file:
@@
 $EndComp
 Text Label 2000 2700 2    50   ~ 0
-RED
+BLUE
 Text Label 2000 2600 2    50   ~ 0
 GREEN
 Text Label 2000 2500 2    50   ~ 0
-BLUE
+RED
 Wire Wire Line
 	2000 2700 2200 2700

Commit message: [design] Add 0ohm resistor for sensor board option
Parts:
- added R4: 0R, symbol Device:R_Small
Connections:
- wire segments 37 -> 40
- no-connect marks 19 -> 18
Other:
- note added: "DNP 0 ohm \nresistor for 5-pin \nsensor board"
Changed lines of the file:
@@
 NoConn ~ 3300 2650
 NoConn ~ 3300 2750
-NoConn ~ 9700 1600
 Wire Wire Line
 	9900 2200 9900 2250
@@
 Wire Wire Line
 	9600 3300 9750 3300
-Text Notes 8400 3550 0    50   ~ 0
+Text Notes 8450 3350 0    50   ~ 0
 Color display for RGB LED:\nNo color: UV Index 0 - 2\nYellow: UV Index 3 - 5\nOrange: UV Index 6 - 7\nRed: UV Index 8 - 10\nPurple: UV Index 11+\n
 $Comp
@@
 Wire Notes Line style solid
 	9000 2750 9000 2550
+$Comp
+L Device:R_Small R4
+U 1 1 5D00B535
+P 9350 1500
+F 0 "R4" V 9300 1350 50  0000 C CNN
+F 1 "0R" V 9400 1350 50  0000 C CNN
+F 2 "" H 9350 1500 50  0001 C CNN
+F 3 "~" H 9350 1500 50  0001 C CNN
+	1    9350 1500
+	0    1    1    0
+$EndComp
+Wire Wire Line
+	9250 1500 9250 1600
+Wire Wire Line
+	9250 1600 9700 1600
+Wire Wire Line
+	9450 1500 9900 1500
+Connection ~ 9900 1500
+Text Notes 8400 1650 0    50   ~ 0
+DNP 0 ohm \nresistor for 5-pin \nsensor board
 $EndSCHEMATC
