File: hardware/Palm.sch (KiCad schematic (older format))
At the start: 11 parts, among them J1 Conn_01x02_Female, Q1 IRLML6402, SW1 SW_SPDT, SW2 SW_SPDT, U1 Adafruit_nRF52_Feather, U2 VEML6075_breakout

Commit message: [bom] Re-generate BOM after adding 1 0R
Parts:
- R4: Category (none) -> Electronics; Package (none) -> 0805; Stock (none) -> 15-res-0805-0
Changed lines of the file:
@@
 F 2 "" H 9350 1500 50  0001 C CNN
 F 3 "~" H 9350 1500 50  0001 C CNN
+F 4 "Electronics" H 0   0   50  0001 C CNN "Category"
+F 5 "0805" H 0   0   50  0001 C CNN "Package"
+F 6 "15-res-0805-0" H 0   0   50  0001 C CNN "Stock"
 	1    9350 1500
 	0    1    1    0

Commit message: [footprint] Generate gerbers
Parts:
- R4: footprint (none) -> Resistor_SMD:R_0805_2012Metric_Pad1.15x1.40mm_HandSolder
Changed lines of the file:
@@
 F 0 "R4" V 9300 1350 50  0000 C CNN
 F 1 "0R" V 9400 1350 50  0000 C CNN
-F 2 "" H 9350 1500 50  0001 C CNN
+F 2 "Resistor_SMD:R_0805_2012Metric_Pad1.15x1.40mm_HandSolder" H 9350 1500 50  0001 C CNN
 F 3 "~" H 9350 1500 50  0001 C CNN
 F 4 "Electronics" H 0   0   50  0001 C CNN "Category"

Commit message: [bom] Update JST PH2 connector body orientation from straight to right angle
Parts:
- J1: footprint Connector_JST:JST_PH_S2B-PH-SM4-TB_1x02-1MP_P2.00mm_Horizontal -> Connector_JST:JST_PH_S2B-PH-SM4-TB_1x02-1MP_P2.00mm_Horizontal, Body orientation: Right angle; Part No. B2B-PH-SM4-TB(LF)(SN) -> S2B-PH-SM4-TB(LF)(SN); Vendor link https://sg.rs-online.com/web/p/pcb-headers/6881325/ -> https://sg.rs-online.com/web/p/products/6881353/
Changed lines of the file:
@@
 F 0 "J1" H 1578 1076 50  0000 L CNN
 F 1 "Conn_01x02_Female" H 1578 985 50  0000 L CNN
-F 2 "Connector_JST:JST_PH_S2B-PH-SM4-TB_1x02-1MP_P2.00mm_Horizontal" H 1550 1100 50  0001 C CNN
-F 3 "https://docs-apac.rs-online.com/webdocs/13ce/0900766b813ce4b4.pdf" H 1550 1100 50  0001 C CNN
+F 2 "Connector_JST:JST_PH_S2B-PH-SM4-TB_1x02-1MP_P2.00mm_Horizontal, Body orientation: Right angle" H 1550 1100 50  0001 C CNN
+F 3 "https://docs-apac.rs-online.com/webdocs/13ce/0900766b813ce4bd.pdf" H 1550 1100 50  0001 C CNN
 F 4 "SMD" H 50  -100 50  0001 C CNN "Package"
 F 5 "RS Components" H 50  -100 50  0001 C CNN "Vendor"
 F 6 "5" H 50  -100 50  0001 C CNN "Minimum Order"
 F 7 "JST" H 200 0   50  0001 C CNN "Manufacturer"
-F 8 "B2B-PH-SM4-TB(LF)(SN) " H 200 0   50  0001 C CNN "Part No."
+F 8 "S2B-PH-SM4-TB(LF)(SN)" H 200 0   50  0001 C CNN "Part No."
 F 9 "0.486" H 200 0   50  0001 C CNN "Unit cost"
-F 10 "https://sg.rs-online.com/web/p/pcb-headers/6881325/" H 200 0   50  0001 C CNN "Vendor link"
+F 10 "https://sg.rs-online.com/web/p/products/6881353/" H 200 0   50  0001 C CNN "Vendor link"
 F 11 "Connector" H 200 0   50  0001 C CNN "Category"
 	1    1550 1100

Commit message: [bom] Add DNP column for BOM and Interactive HTML BOM
Parts:
- R4: DNP (none) -> Yes
Changed lines of the file:
@@
 F 5 "0805" H 0   0   50  0001 C CNN "Package"
 F 6 "15-res-0805-0" H 0   0   50  0001 C CNN "Stock"
+F 7 "Yes" H 0   0   50  0001 C CNN "DNP"
 	1    9350 1500
 	0    1    1    0

Commit message: chore: update submodules with global and project specific symbols and footprints
Parts:
- U1: symbol Adafruit_nRF52_Feather:Adafruit_nRF52_Feather -> Adafruit_nRF52_feather:Adafruit_nRF52_Feather
Changed lines of the file:
@@
 $EndDescr
 $Comp
-L Adafruit_nRF52_Feather:Adafruit_nRF52_Feather U1
+L Adafruit_nRF52_feather:Adafruit_nRF52_Feather U1
 U 1 1 5CB07E1A
 P 2750 2400
